File: M0plus_breakout.brd (EAGLE design)
At the start: 32.5 x 43 mm, 32 parts, among them SW1 SPST_TACT-KMR2, U1 ATSAMD21G-A, U2 SPX3819-3.3, U3 MCP73831T, X1 XTAL_32.768KHZ, X2 microusb

Commit message: added power LED
Parts:
- added LED3: (no value), Ilya_Teach:LED-0603
- added R2: 1k, SparkFun-Resistors:0603
- moved LED2 1.93 mm to (10.9, 12.2)
- moved C9 1.78 mm to (11.6, 20.7)
- moved C10 1.27 mm to (11.6, 15.9)
- moved R1 1.27 mm to (11.7, 14.2)
Connections:
- new net N$7: LED3.C, R2.2
- net 3.3V: now also LED3.A
- net GND: now also R2.1
Routing:
- net 3.3V: track 76.6 -> 82.1 mm
- net D+: track 52.3 -> 56.2 mm
- net D-: track 49.5 -> 51.5 mm
- net N$7: track 0.00 -> 1.80 mm
- net N$5: track 1.54 -> 2.18 mm
Changed lines of the file:
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@@
 <attribute name="VALUE" x="16.764" y="18.415" size="0.4064" layer="27" ratio="10"/>
 </element>
-<element name="C9" library="Ilya_Teach" package="0805" value="10uF" x="11.557" y="18.923" smashed="yes" rot="R180">
-<attribute name="VALUE" x="12.573" y="20.32" size="0.4064" layer="27" rot="R180"/>
-</element>
-<element name="C10" library="Ilya_Teach" package="0805" value="10uF" x="11.5824" y="17.145" smashed="yes" rot="R180">
-<attribute name="VALUE" x="12.5984" y="18.542" size="0.4064" layer="27" rot="R180"/>
+<element name="C9" library="Ilya_Teach" package="0805" value="10uF" x="11.557" y="20.701" smashed="yes" rot="R180">
+<attribute name="VALUE" x="12.573" y="22.098" size="0.4064" layer="27" rot="R180"/>
+</element>
+<element name="C10" library="Ilya_Teach" package="0805" value="10uF" x="11.5824" y="15.875" smashed="yes" rot="R180">
+<attribute name="VALUE" x="12.5984" y="17.272" size="0.4064" layer="27" rot="R180"/>
 </element>
 <element name="U3" library="microbuilder" package="SOT23-5" value="MCP73831T" x="22.86" y="17.526" smashed="yes">
@@
 <attribute name="VALUE" x="16.637" y="18.288" size="0.4064" layer="27" font="vector" rot="R270"/>
 </element>
-<element name="LED2" library="Ilya_Teach" package="LED-0603" value="" x="11.684" y="13.97" smashed="yes" rot="R90">
-<attribute name="VALUE" x="12.7" y="15.0495" size="0.4064" layer="27" rot="R180"/>
-</element>
-<element name="R1" library="SparkFun-Resistors" package="0603-RES" value="1K" x="11.684" y="15.494" smashed="yes" rot="R180">
-<attribute name="PROD_ID" value="RES-07856" x="11.684" y="15.494" size="1.778" layer="27" rot="R180" display="off"/>
-<attribute name="VALUE" x="12.7" y="16.637" size="0.4064" layer="27" font="vector" rot="R180"/>
+<element name="LED2" library="Ilya_Teach" package="LED-0603" value="" x="10.922" y="12.192" smashed="yes" rot="R90">
+<attribute name="VALUE" x="11.938" y="13.2715" size="0.4064" layer="27" rot="R180"/>
+</element>
+<element name="R1" library="SparkFun-Resistors" package="0603-RES" value="1K" x="11.684" y="14.224" smashed="yes" rot="R180">
+<attribute name="PROD_ID" value="RES-07856" x="11.684" y="14.224" size="1.778" layer="27" rot="R180" display="off"/>
+<attribute name="VALUE" x="12.7" y="15.367" size="0.4064" layer="27" font="vector" rot="R180"/>
+</element>
+<element name="LED3" library="Ilya_Teach" package="LED-0603" value="" x="11.43" y="19.05" smashed="yes" rot="R90">
+<attribute name="VALUE" x="12.446" y="20.1295" size="0.4064" layer="27" rot="R180"/>
+</element>
+<element name="R2" library="SparkFun-Resistors" package="0603" value="1k" x="11.684" y="17.526" smashed="yes" rot="R180">
+<attribute name="PROD_ID" value="RES-07856" x="11.684" y="17.526" size="1.778" layer="27" rot="R180" display="off"/>
+<attribute name="VALUE" x="11.684" y="18.288" size="0.6096" layer="27" font="vector" ratio="20" rot="R180" align="top-center"/>
 </element>
 </elements>
@@
 <via x="20.574" y="20.828" extent="1-16" drill="0.4064"/>
 <contactref element="R1" pad="1"/>
+<contactref element="R2" pad="1"/>
 </signal>
 <signal name="N$2">
@@
 <wire x1="19.05" y1="38.354" x2="18.2" y2="38.354" width="0.254" layer="1"/>
 <wire x1="18.2" y1="38.354" x2="18.122" y2="40.132" width="0.254" layer="1"/>
-<wire x1="12.457" y1="18.923" x2="12.5311" y2="20.331" width="0.254" layer="1"/>
-<wire x1="12.5311" y1="20.331" x2="14.036" y2="20.3501" width="0.254" layer="1"/>
 <wire x1="17.692" y1="21.59" x2="16.256" y2="21.59" width="0.254" layer="1"/>
 <wire x1="16.256" y1="21.59" x2="15.24" y2="21.59" width="0.254" layer="1"/>
@@
 <wire x1="19.812" y1="25.654" x2="20.32" y2="25.654" width="0.254" layer="1"/>
 <wire x1="20.32" y1="25.654" x2="20.574" y2="25.4" width="0.254" layer="1"/>
-<wire x1="12.5311" y1="20.331" x2="12.181" y2="20.331" width="0.254" layer="1"/>
-<wire x1="12.181" y1="20.331" x2="11.938" y2="20.574" width="0.254" layer="1"/>
-<via x="11.938" y="20.574" extent="1-16" drill="0.4064"/>
-<wire x1="11.938" y1="20.574" x2="11.938" y2="26.416" width="0.254" layer="16"/>
 <wire x1="11.938" y1="26.416" x2="11.938" y2="33.02" width="0.254" layer="16"/>
 <wire x1="11.938" y1="33.02" x2="11.684" y2="33.274" width="0.254" layer="16"/>
@@
 <wire x1="21.756" y1="20.32" x2="21.706" y2="20.37" width="0.254" layer="1"/>
 <wire x1="21.706" y1="20.37" x2="21.706" y2="21.844" width="0.254" layer="1"/>
+<contactref element="LED3" pad="A"/>
+<wire x1="14.036" y1="20.3501" x2="14.224" y2="20.3501" width="0.4064" layer="1"/>
+<wire x1="14.224" y1="20.3501" x2="14.224" y2="19.05" width="0.4064" layer="1"/>
+<via x="14.224" y="19.05" extent="1-16" drill="0.4064"/>
+<wire x1="14.224" y1="19.05" x2="13.716" y2="19.05" width="0.4064" layer="16"/>
+<wire x1="13.716" y1="19.05" x2="13.716" y2="26.416" width="0.4064" layer="16"/>
+<wire x1="13.716" y1="26.416" x2="11.938" y2="26.416" width="0.4064" layer="16"/>
+<wire x1="12.307" y1="19.05" x2="12.457" y2="19.05" width="0.4064" layer="1"/>
+<wire x1="12.457" y1="19.05" x2="12.457" y2="20.701" width="0.4064" layer="1"/>
+<wire x1="12.457" y1="20.701" x2="14.036" y2="20.701" width="0.4064" layer="1"/>
+<wire x1="14.036" y1="20.701" x2="14.036" y2="20.3501" width="0.4064" layer="1"/>
 </signal>
 <signal name="N$6">
@@
 <wire x1="26.67" y1="38.608" x2="26.67" y2="44.45" width="0.254" layer="1"/>
 <wire x1="26.67" y1="44.45" x2="27.94" y2="45.72" width="0.254" layer="1"/>
-<wire x1="14.732" y1="14.732" x2="14.732" y2="31.75" width="0.254" layer="16"/>
+<wire x1="14.732" y1="21.844" x2="14.732" y2="31.75" width="0.254" layer="16"/>
 <wire x1="14.732" y1="31.75" x2="15.494" y2="32.512" width="0.254" layer="16"/>
 <wire x1="15.494" y1="32.512" x2="17.78" y2="32.512" width="0.254" layer="16"/>
@@
 <wire x1="14.59" y1="10.427" x2="14.59" y2="12.05" width="0.254" layer="1"/>
 <via x="14.732" y="12.954" extent="1-16" drill="0.4064"/>
-<wire x1="14.732" y1="12.954" x2="15.24" y2="13.716" width="0.254" layer="16"/>
-<wire x1="15.24" y1="13.716" x2="15.24" y2="14.224" width="0.254" layer="16"/>
-<wire x1="15.24" y1="14.224" x2="14.732" y2="14.732" width="0.254" layer="16"/>
+<wire x1="14.732" y1="12.954" x2="16.51" y2="13.716" width="0.254" layer="16"/>
+<wire x1="16.51" y1="13.716" x2="16.51" y2="21.082" width="0.254" layer="16"/>
+<wire x1="16.51" y1="21.082" x2="14.732" y2="21.844" width="0.254" layer="16"/>
 <wire x1="14.59" y1="12.05" x2="14.732" y2="12.192" width="0.254" layer="1"/>
 <wire x1="14.732" y1="12.192" x2="14.732" y2="12.954" width="0.254" layer="1"/>
@@
 <wire x1="15.494" y1="13.716" x2="14.224" y2="13.716" width="0.254" layer="1"/>
 <via x="14.224" y="13.716" extent="1-16" drill="0.4064"/>
-<wire x1="14.224" y1="13.716" x2="14.224" y2="32.004" width="0.254" layer="16"/>
+<wire x1="14.224" y1="13.716" x2="16.002" y2="13.97" width="0.254" layer="16"/>
+<wire x1="16.002" y1="13.97" x2="16.002" y2="20.828" width="0.254" layer="16"/>
+<wire x1="16.002" y1="20.828" x2="14.224" y2="21.59" width="0.254" layer="16"/>
+<wire x1="14.224" y1="21.59" x2="14.224" y2="32.004" width="0.254" layer="16"/>
 <wire x1="14.224" y1="32.004" x2="15.24" y2="33.02" width="0.254" layer="16"/>
 <wire x1="15.24" y1="33.02" x2="18.034" y2="33.02" width="0.254" layer="16"/>
@@
 <wire x1="24.288" y1="33.02" x2="24.316" y2="32.992" width="0.254" layer="1"/>
 <contactref element="LED2" pad="A"/>
-<wire x1="14.224" y1="13.716" x2="13.462" y2="13.97" width="0.254" layer="1"/>
-<wire x1="13.462" y1="13.97" x2="12.561" y2="13.97" width="0.254" layer="1"/>
+<wire x1="14.224" y1="13.716" x2="12.7" y2="12.7" width="0.254" layer="1"/>
+<wire x1="12.7" y1="12.7" x2="11.799" y2="12.192" width="0.254" layer="1"/>
 </signal>
 <signal name="AREF">
@@
 <wire x1="22.86" y1="18.288" x2="22.86" y2="18.034" width="0.254" layer="1"/>
 <wire x1="22.86" y1="18.034" x2="22.1996" y2="17.3736" width="0.254" layer="1"/>
-<wire x1="14.136" y1="15.494" x2="14.136" y2="17.6499" width="0.254" layer="1"/>
+<wire x1="14.136" y1="15.494" x2="14.136" y2="16.002" width="0.254" layer="1"/>
+<wire x1="14.136" y1="16.002" x2="14.136" y2="17.6499" width="0.254" layer="1"/>
 <wire x1="14.136" y1="17.6499" x2="14.036" y2="17.7499" width="0.254" layer="1"/>
-<wire x1="14.036" y1="17.7499" x2="12.9951" y2="17.7499" width="0.254" layer="1"/>
-<wire x1="12.9951" y1="17.7499" x2="12.4824" y2="17.145" width="0.254" layer="1"/>
 <wire x1="17.78" y1="16.422" x2="17.946" y2="16.676" width="0.254" layer="1"/>
 <wire x1="17.946" y1="16.676" x2="17.526" y2="16.256" width="0.254" layer="1"/>
@@
 <via x="17.272" y="12.954" extent="1-16" drill="0.4064"/>
 <wire x1="17.272" y1="12.954" x2="17.272" y2="14.478" width="0.4064" layer="1"/>
+<wire x1="12.4824" y1="15.875" x2="14.136" y2="15.875" width="0.4064" layer="1"/>
+<wire x1="14.136" y1="15.875" x2="14.136" y2="16.002" width="0.4064" layer="1"/>
 </signal>
 <signal name="V_BATT">
@@
 <contactref element="LED2" pad="C"/>
 <contactref element="R1" pad="2"/>
-<wire x1="10.807" y1="13.97" x2="10.834" y2="13.997" width="0.254" layer="1"/>
-<wire x1="10.834" y1="13.997" x2="10.834" y2="15.494" width="0.254" layer="1"/>
+<wire x1="10.045" y1="12.192" x2="10.326" y2="12.981" width="0.254" layer="1"/>
+<wire x1="10.326" y1="12.981" x2="10.834" y2="14.224" width="0.254" layer="1"/>
+</signal>
+<signal name="N$7">
+<contactref element="R2" pad="2"/>
+<contactref element="LED3" pad="C"/>
+<wire x1="10.553" y1="19.05" x2="10.834" y2="19.05" width="0.4064" layer="1"/>
+<wire x1="10.834" y1="19.05" x2="10.834" y2="17.526" width="0.4064" layer="1"/>
 </signal>
 </signals>
